File: kicad/analog.kicad_sch (KiCad schematic)
At the start: 0 parts

Commit message: add charging/balancing IC to library
Parts:
- added U1: MP2672GD-0000-Z, 4in-power:QFN-18_2MMx3MM_MP2672_MNP_MPS, symbol 4in-power:MP2672GD-0000-Z
Changed lines of the file:
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@@
 	(generator_version "9.0")
 	(paper "A4")
+	(symbol
+		(lib_id "4in-power:MP2672GD-0000-Z")
+		(at 106.68 60.96 0)
+		(unit 1)
+		(exclude_from_sim no)
+		(in_bom yes)
+		(on_board yes)
+		(dnp no)
+		(fields_autoplaced yes)
+		(property "Reference" "U1"
+			(at 127 50.8 0)
+			(effects
+				(font
+					(size 1.524 1.524)
+				)
+			)
+		)
+		(property "Value" "MP2672GD-0000-Z"
+			(at 127 53.34 0)
+			(effects
+				(font
+					(size 1.524 1.524)
+				)
+			)
+		)
+		(property "Footprint" "4in-power:QFN-18_2MMx3MM_MP2672_MNP_MPS"
+			(at 106.68 60.96 0)
+			(effects
+				(font
+					(size 1.27 1.27)
+					(italic yes)
+				)
+				(hide yes)
+			)
+		)
+		(property "Datasheet" "https://www.monolithicpower.com/en/documentview/productdocument/index/version/2/document_type/Datasheet/lang/en/sku/MP2672"
+			(at 106.68 60.96 0)
+			(effects
+				(font
+					(size 1.27 1.27)
+					(italic yes)
+				)
+				(hide yes)
+			)
+		)
+		(property "Description" "Charging/Balancing IC"
+			(at 106.68 60.96 0)
+			(effects
+				(font
+					(size 1.27 1.27)
+				)
+				(hide yes)
+			)
+		)
+		(property "Manufacturer PN" "MP2672GD-0000-P"
+			(at 106.68 60.96 0)
+			(effects
+				(font
+					(size 1.27 1.27)
+				)
+				(hide yes)
+			)
+		)
+		(property "LCSC PN " "C2837210"
+			(at 106.68 60.96 0)
+			(effects
+				(font
+					(size 1.27 1.27)
+				)
+				(hide yes)
+			)
+		)
+		(property "DigKey Link" "https://www.digikey.ca/en/products/detail/monolithic-power-systems-inc/MP2672GD-0000-Z/13159530"
+			(at 106.68 60.96 0)
+			(effects
+				(font
+					(size 1.27 1.27)
+				)
+				(hide yes)
+			)
+		)
+		(property "JLC Price" "3.6991"
+			(at 106.68 60.96 0)
+			(effects
+				(font
+					(size 1.27 1.27)
+				)
+				(hide yes)
+			)
+		)
+		(pin "15"
+		)
+		(pin "8"
+		)
+		(pin "18"
+		)
+		(pin "17"
+		)
+		(pin "13"
+		)
+		(pin "14"
+		)
+		(pin "16"
+		)
+		(pin "9"
+		)
+		(pin "7"
+		)
+		(pin "6"
+		)
+		(pin "5"
+		)
+		(pin "4"
+		)
+		(pin "1"
+		)
+		(pin "2"
+		)
+		(pin "3"
+		)
+		(pin "10"
+		)
+		(pin "12"
+		)
+		(pin "11"
+		)
+		(instances
+			(project ""
+				(path "/612ece3f-e722-4b33-8111-645d24cfcf05/b5ab9921-5796-498c-b0d6-2d1294fdeff4"
+					(reference "U1")
+					(unit 1)
+				)
+			)
+		)
+	)
 )

Commit message: add new ICs to library
Parts:
- added BT1, BT2: Battery_Cell, symbol Device:Battery_Cell
- added C1, C4, C5, C6, C9: 22u, Capacitor_SMD:C_0402_1005Metric, symbol Device:C
- added C12, C13, C17, C18, C19, C22: 22u, Capacitor_SMD:C_0805_2012Metric, symbol Device:C
- added C14: 1u, Capacitor_SMD:C_0805_2012Metric, symbol Device:C
- added C15, C23: 1u, Capacitor_SMD:C_0603_1608Metric, symbol Device:C
- added C16: 0.1u, Capacitor_SMD:C_0603_1608Metric, symbol Device:C
- added C2: 220p, Capacitor_SMD:C_0402_1005Metric, symbol Device:C
- added C20: 220p, Capacitor_SMD:C_0603_1608Metric, symbol Device:C
- added C21: 10u, Capacitor_SMD:C_0805_2012Metric, symbol Device:C
- added C24, C27, C28, C29: C, symbol Device:C
- added C25: 22u, Capacitor_SMD:C_1206_3216Metric, symbol Device:C
- added C26: 100n, Capacitor_SMD:C_0603_1608Metric, symbol Device:C
- added C3: 0.1u, Capacitor_SMD:C_0402_1005Metric, symbol Device:C
- added C7, C8: 1u, Capacitor_SMD:C_0402_1005Metric, symbol Device:C
- added D3, D4: LED, LED_SMD:LED_0603_1608Metric, symbol Device:LED
- added L1: MPL-AL6050-3R3, POWERLIB:2-SMD, symbol Device:L
- added L2: MPL-AL6050-2R2, POWERLIB:2-SMD, symbol Device:L
- added L3: 1.5uH, POWERLIB:IND-SMD_L7.0-W6.6, symbol powermodule:MWSA0605S-1R5MT
- added L4: L, symbol Device:L
- added R1: 22.1k, Resistor_SMD:R_0603_1608Metric, symbol Device:R
- added R10: 100k, Resistor_SMD:R_0402_1005Metric, symbol Device:R
- added R11: 10R, Resistor_SMD:R_1206_3216Metric, symbol Device:R
- added R13: 100k, Resistor_SMD:R_0603_1608Metric, symbol Device:R
- added R14: 5.5k, Resistor_SMD:R_0603_1608Metric, symbol Device:R
- added R15, R24: 100R, Resistor_SMD:R_0805_2012Metric, symbol Device:R
- added R16: 30k, Resistor_SMD:R_0603_1608Metric, symbol Device:R
- added R17, R23: 60R, Resistor_SMD:R_1206_3216Metric, symbol Device:R
- added R18: 8k, Resistor_SMD:R_0603_1608Metric, symbol Device:R
- added R19: 12.6k, Resistor_SMD:R_0603_1608Metric, symbol Device:R
- added R20: 3.6k, Resistor_SMD:R_0603_1608Metric, symbol Device:R
- added R21: 2k, Resistor_SMD:R_0603_1608Metric, symbol Device:R
- added R22: NTCG103JF103FT1, Diode_SMD:D_0402_1005Metric, symbol powermodule:NTCG103JF103FT1
- added R25, R5, R6, R7: R, symbol Device:R
- added R8: 10R, Resistor_SMD:R_0402_1005Metric, symbol Device:R
- added R9: 13.7k, Resistor_SMD:R_0402_1005Metric, symbol Device:R
- added U3: MP2236CGJ-Z, TSOT23-8_MP2236C_MNP, symbol 4in-power:MP2236CGJ-Z
- added U5: MP2672GD-0000-Z, POWERLIB:QFN-18_2MMx3MM_MP2672_MNP_MPS, symbol powermodule:MP2672GD-0000-Z
- added U6, U7: MP2236CGJ-P, POWERLIB:TSOT23-8_MP2236C_MNP, symbol powermodule:MP2236CGJ-P
Connections:
- net VBUS: now reaches U1.1 (IN)
- net VBUS: now also C27.2, L4.1, R5.1
- net at U1.10 (BATT): now also BT1.1 (+)
- net at U1.11 (SYS): now also C29.1
- net GND: now reaches U1.13 (PGND)
- net GND: now also BT2.2 (-), C29.2, R6.2, R7.2
- net VCC: now reaches U1.16 (*STAT)
- net VCC: now also U1.18 (*ACOK), U1.8 (NTC), C23.1, R15.1, R19.1, R24.1, U5.4 (VCC)
- net at U1.17 (CV): now also R25.1
- net at U1.2 (SW): now also C24.1, L4.2
- net at U1.3 (BST): now also C24.2
- net at U1.4 (VCC): now also C28.1
- net at U1.5 (ISET): now also R7.1
- net AGND: now reaches U1.6 (AGND)
- net AGND: now also C28.2, R25.2
- net at U1.7 (VLIM): now also R5.2, R6.1
- net at U1.9 (MID): now also BT1.2 (-), BT2.1 (+)
- new net: C26.2, U5.3 (BST)
- new net: R17.1, R23.1, U5.9 (MID)
- new net: R20.1, R22.2
- new net: D4.2 (A), R24.2
- new net: R8.2, U7.5 (BST)
- new net: C7.2, U7.7 (VCC)
- new net: C3.1, R8.1
- new net: C15.2, U6.7 (VCC)
- new net: R18.1, U5.5 (ISET)
- new net: R19.2, R20.2, U5.8 (NTC)
- new net: C22.2, U5.11 (SYS)
- new net: D4.1 (K), U5.16 (*STAT)
- new net: R16.1, U5.17 (CV)
- new net: D3.1 (K), U5.18 (*ACOK)
- new net: R11.2, U6.5 (BST)
- new net: D3.2 (A), R15.2
- new net: C16.1, R11.1
- new net +3.3V OUT: C17.1, C18.1, C19.1, C20.1, L2.2, R13.2
- new net +4.2V: R17.2, R23.2
- new net +5V OUT: C2.1, C4.1, C5.1, C6.1, L1.2, R10.2
- new net +8.4V: C1.2, C12.2, C13.2, C14.1, C25.1, C8.1, C9.2, U5.10 (BATT), U6.2 (IN), U7.2 (IN)
- new net EN1: U7.6 (EN)
- new net EN2: U6.6 (EN)
- new net FB1: C2.2, R10.1, R9.2, U7.8 (FB)
- new net FB2: C20.2, R1.2, R13.1, U6.8 (FB)
- new net L3P2: C26.1, L3.2, U5.2 (SW)
- new net LOAD_GND: C1.1, C12.1, C13.1, C14.2, C15.1, C17.2, C18.2, C19.2, C21.2, C22.1, C23.2, C25.2, C4.2, C5.2, C6.2, C7.1, C8.2, C9.1, R1.1, R16.2, R18.2, R21.1, R22.1, R9.1, U5.13 (PGND), U5.6 (AGND), U6.1 (AGND), U6.4 (GND), U7.1 (AGND), U7.4 (GND)
- new net SCL: U5.14 (SCL)
- new net SDA: U5.15 (SDA)
- new net SW1: C3.2, L1.1, U7.3 (SW)
- new net SW2: C16.2, L2.1, U6.3 (SW)
- new net VIN: C21.1, L3.1, R14.2, U5.1 (IN)
- new net VLIM: R14.1, R21.2, U5.7 (VLIM)
- no-connect marks 0 -> 3
Other:
- note added: "- get fuel guage for next version"
- note added: "Charging and Balancing"
- note added: "Step down 5v to 3.3v"
- note added: "Step down 8.4v to 5v"
