File: kicad/analog.kicad_sch (KiCad schematic)
At the start: 42 parts, among them U402 MP2672GD-0000-Z, U403 Battery, U501 TPS63070RNMR, U601 TPS63070RNMR

Commit message: complete BOM
Parts:
- C406, C501, C502, C503, C505, C601, C602, C607, C608: footprint (none) -> 1206; JLC Link (none) -> https://jlcpcb.com/partdetail/2201-CL31A106KOHNNNE/C1849; LCSC PN (none) -> C1849
- C408, C409, C506, C507, C508, C604, C605, C606: footprint (none) -> 1206; JLC Link (none) -> https://jlcpcb.com/partdetail/2211-1206X226K100NT/C1859; LCSC PN (none) -> C1859
- R404: JLC Link (none) -> https://jlcpcb.com/partdetail/Ever_OhmsTech-TR0805B25K0P052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; LCSC PN (none) -> C153306
- R408: footprint (none) -> 0603; JLC Link (none) -> https://jlcpcb.com/partdetail/4623-0603WAF3302T5E/C4216; LCSC PN (none) -> C4216
- R409: footprint (none) -> 0805
- R502: footprint (none) -> 0805; JLC Link (none) -> https://jlcpcb.com/partdetail/18397-0805W8F4703T5E/C17709; LCSC PN (none) -> C17709
- R503: footprint (none) -> 0402; JLC Link (none) -> https://jlcpcb.com/partdetail/1518-RS02K154JT/C1166; LCSC PN (none) -> C1166
- R504, R602: footprint (none) -> 1206; JLC Link (none) -> https://jlcpcb.com/partdetail/18588-1206W4F1003T5E/C17900; LCSC PN (none) -> C17900
Other:
- note removed: "double check these resistors"
- moved on the sheet: R404

Commit message: add all components to schematic
Parts:
- C406, C408, C409, C501, C502, C503, C505, C506, C507, C508, C601, C602, C604, C605, C606, C607, C608: footprint 1206 -> Capacitor_SMD:C_1206_3216Metric
- R408: footprint 0603 -> Resistor_SMD:R_0603_1608Metric
- R409, R502: footprint 0805 -> Resistor_SMD:R_0805_2012Metric
- R503: footprint 0402 -> Resistor_SMD:R_0402_1005Metric
- R504, R602: footprint 1206 -> Resistor_SMD:R_1206_3216Metric
Changed lines of the file:
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@@
 			)
 		)
-		(property "Footprint" "1206"
+		(property "Footprint" "Capacitor_SMD:C_1206_3216Metric"
 			(at 260.0452 73.66 0)
 			(effects
@@
 			)
 		)
-		(property "Footprint" "1206"
+		(property "Footprint" "Capacitor_SMD:C_1206_3216Metric"
 			(at 141.2748 45.72 0)
 			(effects
@@
 			)
 		)
-		(property "Footprint" "1206"
+		(property "Footprint" "Capacitor_SMD:C_1206_3216Metric"
 			(at 36.5252 182.88 0)
 			(effects
@@
 			)
 		)
-		(property "Footprint" "1206"
+		(property "Footprint" "Capacitor_SMD:C_1206_3216Metric"
 			(at 196.5452 181.61 0)
 			(effects
@@
 			)
 		)
-		(property "Footprint" "0603"
+		(property "Footprint" "Resistor_SMD:R_0603_1608Metric"
 			(at 90.932 91.44 90)
 			(effects
@@
 			)
 		)
-		(property "Footprint" "1206"
+		(property "Footprint" "Capacitor_SMD:C_1206_3216Metric"
 			(at 373.0752 72.39 0)
 			(effects
@@
 			)
 		)
-		(property "Footprint" "1206"
+		(property "Footprint" "Capacitor_SMD:C_1206_3216Metric"
 			(at 361.6452 72.39 0)
 			(effects
@@
 			)
 		)
-		(property "Footprint" "1206"
+		(property "Footprint" "Capacitor_SMD:C_1206_3216Metric"
 			(at 149.5552 181.61 0)
 			(effects
@@
 			)
 		)
-		(property "Footprint" "0805"
+		(property "Footprint" "Resistor_SMD:R_0805_2012Metric"
 			(at 333.502 68.58 90)
 			(effects
@@
 			)
 		)
-		(property "Footprint" "1206"
+		(property "Footprint" "Resistor_SMD:R_1206_3216Metric"
 			(at 350.012 83.82 90)
 			(effects
@@
 			)
 		)
-		(property "Footprint" "1206"
+		(property "Footprint" "Capacitor_SMD:C_1206_3216Metric"
 			(at 47.9552 182.88 0)
 			(effects
@@
 			)
 		)
-		(property "Footprint" "1206"
+		(property "Footprint" "Capacitor_SMD:C_1206_3216Metric"
 			(at 79.7052 182.88 0)
 			(effects
@@
 			)
 		)
-		(property "Footprint" "1206"
+		(property "Footprint" "Resistor_SMD:R_1206_3216Metric"
 			(at 162.052 193.04 90)
 			(effects
@@
 			)
 		)
-		(property "Footprint" "0805"
+		(property "Footprint" "Resistor_SMD:R_0805_2012Metric"
 			(at 102.362 97.79 90)
 			(effects
@@
 			)
 		)
-		(property "Footprint" "1206"
+		(property "Footprint" "Capacitor_SMD:C_1206_3216Metric"
 			(at 32.0548 64.77 0)
 			(effects
@@
 			)
 		)
-		(property "Footprint" "1206"
+		(property "Footprint" "Capacitor_SMD:C_1206_3216Metric"
 			(at 173.6852 181.61 0)
 			(effects
@@
 			)
 		)
-		(property "Footprint" "1206"
+		(property "Footprint" "Capacitor_SMD:C_1206_3216Metric"
 			(at 384.5052 72.39 0)
 			(effects
@@
 			)
 		)
-		(property "Footprint" "0402"
+		(property "Footprint" "Resistor_SMD:R_0402_1005Metric"
 			(at 333.502 76.2 90)
 			(effects
@@
 			)
 		)
-		(property "Footprint" "1206"
+		(property "Footprint" "Capacitor_SMD:C_1206_3216Metric"
 			(at 230.8352 73.66 0)
 			(effects
@@
 			)
 		)
-		(property "Footprint" "1206"
+		(property "Footprint" "Capacitor_SMD:C_1206_3216Metric"
 			(at 219.4052 73.66 0)
 			(effects
@@
 			)
 		)
-		(property "Footprint" "1206"
+		(property "Footprint" "Capacitor_SMD:C_1206_3216Metric"
 			(at 152.7048 45.72 0)
 			(effects
@@
 			)
 		)
-		(property "Footprint" "1206"
+		(property "Footprint" "Capacitor_SMD:C_1206_3216Metric"
 			(at 318.4652 72.39 0)
 			(effects
@@
 			)
 		)
-		(property "Footprint" "1206"
+		(property "Footprint" "Capacitor_SMD:C_1206_3216Metric"
 			(at 185.1152 181.61 0)
 			(effects

Commit message: progress charging/balancing routing
Parts:
- U403: value Battery -> Battery (MR-30)
Changed lines of the file:
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@@
 		(on_board yes)
 		(dnp no)
-		(fields_autoplaced yes)
 		(property "Reference" "U403"
-			(at 185.42 69.8499 0)
+			(at 184.912 72.898 0)
 			(effects
 				(font
@@
 			)
 		)
-		(property "Value" "Battery"
-			(at 185.42 72.3899 0)
+		(property "Value" "Battery (MR-30)"
+			(at 179.07 77.724 0)
 			(effects
 				(font

Commit message: start via stitching
Connections:
- net VCC: now also C410.2, U402.4 (VCC)
Changed lines of the file:
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@@
+		)
+	)
+	(label "VCC"
+		(at 153.67 77.47 0)
+		(effects
+			(font
+				(size 1.27 1.27)
+			)
+			(justify left bottom)
 		)
 	)

Commit message: export final production files for 0.1.0
Parts:
- added C430: 22u, Capacitor_SMD:C_1206_3216Metric, symbol Device:C
- added R460, R461: 33m, Resistor_SMD:R_1206_3216Metric, symbol Device:R
- R503: footprint Resistor_SMD:R_0402_1005Metric -> Resistor_SMD:R_0805_2012Metric; JLC Link https://jlcpcb.com/partdetail/1518-RS02K154JT/C1166 -> https://jlcpcb.com/partdetail/18158-0805W8F1503T5E/C17470; LCSC PN C1166 -> C17470
Connections:
- net GND: now also C430.1
- net at U402.10 (BATT), U403.1: now also C430.2
- net at U402.9 (MID): now also R460.1, R461.1; no longer U403.2
- new net: R460.2, R461.2, U403.2
Other:
- moved on the sheet: C408, C409, C410
