File: kicad/Power.kicad_sch (KiCad schematic)
At the start: 10 parts

Commit message: Wrong Commit lmao
Parts:
- added J1, J2, J3, J4, J5: Conn_01x02, symbol Connector_Generic:Conn_01x02
- renumbered C19 to C18, C20 to C19, C21 to C20, C22 to C21, R15 to R10, R16 to R11, R17 to R12, R18 to R13, R19 to R14, R14 to R9
Connections:
- net GND: now also J1.1 (Pin_1), J2.1 (Pin_1), J3.1 (Pin_1), J4.2 (Pin_2), J5.2 (Pin_2)
- new net ServoReg1/SERVO_PWR: J4.1 (Pin_1)
- new net ServoReg2/SERVO_PWR: J5.1 (Pin_1)
- new net UNREG_PWR: J1.2 (Pin_2), J2.2 (Pin_2), J3.2 (Pin_2)
Other:
- removed sheet Battery
- removed sheet Boost24V
- removed sheet Charger
- added sheet Power Input (PowerInput.kicad_sch)
- added sheet ServoReg1 (ServoReg.kicad_sch)
- added sheet ServoReg2 (ServoReg.kicad_sch)
- note added: "2A RATING"
- note added: "3A RATING"
- note added: "Unregulated Output"
- note removed: "5V Buck-boost"
- title: Power Interconnects -> (none)
- moved on the sheet: C18, C19, C20, C21, R10, R11, R12, R13, R14, R9
